File: Keyboard Matrix.sch (KiCad schematic (older format))
At the start: 83 parts

Commit message: update to kicad schematic and pcb
Parts:
- removed D? (x2): D_Small, symbol Device:D_Small
- added D10, D11, D12, D13, D14, D15, D16, D17, D18, D19, D20, D21, D22, D23, D24, D25, D26, D27, D28, D29, D30, D31, D32, D33, D34, D35, D36, D37, D38, D39, D4, D40, D41, D42, D43, D44, D45, D46, D47, D48, D49, D5, D50, D51, D52, D53, D54, D55, D56, D57, D58, D59, D6, D60, D61, D62, D63, D64, D65, D66, D67, D68, D69, D7, D70, D71, D72, D73, D74, D75, D76, D77, D78, D79, D8, D80, D81, D82, D83, D9: 1N4148TR, Diode_THT:D_DO-35_SOD27_P7.62mm_Horizontal, symbol Device:D_Small
- D3: renamed from D?; value D_Small -> 1N4148TR; footprint (none) -> Diode_THT:D_DO-35_SOD27_P7.62mm_Horizontal
- MX10: renamed from MX?; value MX-NoLED -> A
- MX11: renamed from MX?; value MX-NoLED -> Z
- MX12: renamed from MX?; value MX-NoLED -> Alt
- MX15: renamed from MX?; value MX-NoLED -> W
- MX16: renamed from MX?; value MX-NoLED -> S
- MX17: renamed from MX?; value MX-NoLED -> X
- MX19: renamed from MX?; value MX-NoLED -> E
- MX20: renamed from MX?; value MX-NoLED -> D
- MX21: renamed from MX?; value MX-NoLED -> C
- MX24: renamed from MX?; value MX-NoLED -> R
- MX25: renamed from MX?; value MX-NoLED -> F
- MX26: renamed from MX?; value MX-NoLED -> V
- MX29: renamed from MX?; value MX-NoLED -> T
- MX3: renamed from MX?; value MX-NoLED -> Tab
- MX30: renamed from MX?; value MX-NoLED -> G
- MX31: renamed from MX?; value MX-NoLED -> B
- MX34: renamed from MX?; value MX-NoLED -> Y
- MX35: renamed from MX?; value MX-NoLED -> H
- MX36: renamed from MX?; value MX-NoLED -> N
- MX39: renamed from MX?; value MX-NoLED -> U
- MX4: renamed from MX?; value MX-NoLED -> Step Caps
- MX40: renamed from MX?; value MX-NoLED -> J
- MX41: renamed from MX?; value MX-NoLED -> M
- MX44: renamed from MX?; value MX-NoLED -> I
- MX45: renamed from MX?; value MX-NoLED -> K
- MX46: renamed from MX?; value MX-NoLED -> <
- MX47: renamed from MX?; value MX-NoLED -> R Alt
- MX5: renamed from MX?; value MX-NoLED -> Shift
- MX50: renamed from MX?; value MX-NoLED -> O
- MX51: renamed from MX?; value MX-NoLED -> L
- MX52: renamed from MX?; value MX-NoLED -> >
- MX55: renamed from MX?; value MX-NoLED -> P
- MX56: renamed from MX?; value MX-NoLED -> ;
- MX57: renamed from MX?; value MX-NoLED -> /
- MX58: renamed from MX?; value MX-NoLED -> R Ctrl
- MX6: renamed from MX?; value MX-NoLED -> Ctrl
- MX61: renamed from MX?; value MX-NoLED -> [
- MX62: renamed from MX?; value MX-NoLED -> '
- MX63: renamed from MX?; value MX-NoLED -> RShift
- MX64: renamed from MX?; value MX-NoLED -> Left Arrow
- MX67: renamed from MX?; value MX-NoLED -> ]
- MX68: renamed from MX?; value MX-NoLED -> Enter
- MX71: renamed from MX?; value MX-NoLED -> bACKSPACE
- MX73: renamed from MX?; value MX-NoLED -> Up Arrow
- MX74: renamed from MX?; value MX-NoLED -> Down Arrow
- MX77: renamed from MX?; value MX-NoLED -> PgUp
- MX78: renamed from MX?; value MX-NoLED -> PgDn
- MX79: renamed from MX?; value MX-NoLED -> End
- MX80: renamed from MX?; value MX-NoLED -> Right Arrow
- MX9: renamed from MX?; value MX-NoLED -> Q
- gave numbers to parts that had none: 30
Connections:
- net Row_0: now also D15.1 (K), D24.1 (K), D35.1 (K), D45.1 (K), D56.1 (K), D68.1 (K), D78.1 (K)
- net Row_1: now also D29.1 (K), D40.1 (K), D51.1 (K), D62.1 (K), D72.1 (K), D9.1 (K)
- net Col_0: now reaches MX1.1 (COL)
- net Col_0: now also MX10.1 (COL), MX11.1 (COL), MX12.1 (COL), MX2.1 (COL), MX3.1 (COL), MX4.1 (COL), MX5.1 (COL), MX6.1 (COL), MX7.1 (COL), MX8.1 (COL), MX9.1 (COL)
- net at MX7.2 (ROW): now also D9.2 (A)
- net Col_1: now reaches MX13.1 (COL)
- net Col_1: now also MX14.1 (COL), MX15.1 (COL), MX16.1 (COL), MX17.1 (COL), MX18.1 (COL), MX19.1 (COL), MX20.1 (COL), MX21.1 (COL)
- net at MX13.2 (ROW): now also D15.2 (A)
- net Col_2: now reaches MX22.1 (COL)
- net Col_2: now also MX23.1 (COL), MX24.1 (COL), MX25.1 (COL), MX26.1 (COL), MX27.1 (COL), MX28.1 (COL), MX29.1 (COL), MX30.1 (COL), MX31.1 (COL)
- net at MX22.2 (ROW): now also D24.2 (A)
- net at MX27.2 (ROW): now also D29.2 (A)
- net Col_3: now reaches MX32.1 (COL)
- net Col_3: now also MX33.1 (COL), MX34.1 (COL), MX35.1 (COL), MX36.1 (COL), MX37.1 (COL), MX38.1 (COL), MX39.1 (COL), MX40.1 (COL), MX41.1 (COL)
- net at MX32.2 (ROW): now also D35.2 (A)
- net at MX37.2 (ROW): now also D40.2 (A)
- net Col_4: now reaches MX42.1 (COL)
- net Col_4: now also MX43.1 (COL), MX44.1 (COL), MX45.1 (COL), MX46.1 (COL), MX47.1 (COL), MX48.1 (COL), MX49.1 (COL), MX50.1 (COL), MX51.1 (COL), MX52.1 (COL)
- net at MX42.2 (ROW): now also D45.2 (A)
- net at MX48.2 (ROW): now also D51.2 (A)
- net Col_5: now reaches MX53.1 (COL)
- net Col_5: now also MX54.1 (COL), MX55.1 (COL), MX56.1 (COL), MX57.1 (COL), MX58.1 (COL), MX59.1 (COL), MX60.1 (COL), MX61.1 (COL), MX62.1 (COL), MX63.1 (COL), MX64.1 (COL)
- net at MX53.2 (ROW): now also D56.2 (A)
- net at MX59.2 (ROW): now also D62.2 (A)
- net Col_6: now reaches MX65.1 (COL)
- net Col_6: now also MX66.1 (COL), MX67.1 (COL), MX68.1 (COL), MX69.1 (COL), MX70.1 (COL), MX71.1 (COL), MX73.1 (COL), MX74.1 (COL), MX78.1 (COL), MX79.1 (COL), MX80.1 (COL)
- net at MX65.2 (ROW): now also D68.2 (A)
- net at MX69.2 (ROW): now also D72.2 (A)
- net Col_7: now reaches MX75.1 (COL)
- net Col_7: now also MX72.1 (COL), MX76.1 (COL), MX77.1 (COL)
- net at MX75.2 (ROW): now also D78.2 (A)
- net at MX2.2 (ROW): now also D4.2 (A)
- net at MX8.2 (ROW): now also D10.2 (A)
- net at MX14.2 (ROW): now also D16.2 (A)
- net at MX18.2 (ROW): now also D20.2 (A)
- net at MX23.2 (ROW): now also D25.2 (A)
- net at MX28.2 (ROW): now also D30.2 (A)
- net at MX33.2 (ROW): now also D36.2 (A)
- net at MX38.2 (ROW): now also D41.2 (A)
- net at MX43.2 (ROW): now also D46.2 (A)
- net at MX49.2 (ROW): now also D52.2 (A)
- net at MX54.2 (ROW): now also D57.2 (A)
- net at MX60.2 (ROW): now also D63.2 (A)
- net at MX66.2 (ROW): now also D69.2 (A)
- net at MX70.2 (ROW): now also D73.2 (A)
- net at MX72.2 (ROW): now also D75.2 (A)
- net at MX76.2 (ROW): now also D79.2 (A)
- net at MX9.2 (ROW): now also D11.2 (A)
- net at MX15.2 (ROW): now also D17.2 (A)
- net at MX19.2 (ROW): now also D21.2 (A)
- net at MX24.2 (ROW): now also D26.2 (A)
- net at MX29.2 (ROW): now also D31.2 (A)
- net at MX34.2 (ROW): now also D37.2 (A)
- net at MX39.2 (ROW): now also D42.2 (A)
- net at MX44.2 (ROW): now also D47.2 (A)
- net at MX50.2 (ROW): now also D53.2 (A)
- net at MX55.2 (ROW): now also D58.2 (A)
- net at MX61.2 (ROW): now also D64.2 (A)
- net at MX67.2 (ROW): now also D70.2 (A)
- net at MX77.2 (ROW): now also D80.2 (A)
- net at MX10.2 (ROW): now also D12.2 (A)
- net at MX16.2 (ROW): now also D18.2 (A)
- net at MX20.2 (ROW): now also D22.2 (A)
- net at MX25.2 (ROW): now also D27.2 (A)
- net at MX30.2 (ROW): now also D32.2 (A)
- net at MX35.2 (ROW): now also D38.2 (A)
- net at MX40.2 (ROW): now also D43.2 (A)
- net at MX45.2 (ROW): now also D48.2 (A)
- net at MX51.2 (ROW): now also D54.2 (A)
- net at MX56.2 (ROW): now also D59.2 (A)
- net at MX62.2 (ROW): now also D65.2 (A)
- net at MX78.2 (ROW): now also D81.2 (A)
- net at MX11.2 (ROW): now also D13.2 (A)
- net at MX12.2 (ROW): now also D14.2 (A)
- net at MX17.2 (ROW): now also D19.2 (A)
- net at MX21.2 (ROW): now also D23.2 (A)
- net at MX26.2 (ROW): now also D28.2 (A)
- net at MX31.2 (ROW): now also D33.2 (A)
- net at MX36.2 (ROW): now also D39.2 (A)
- net at MX41.2 (ROW): now also D44.2 (A)
- net at MX46.2 (ROW): now also D49.2 (A)
- net at MX47.2 (ROW): now also D50.2 (A)
- net at MX52.2 (ROW): now also D55.2 (A)
- net at MX57.2 (ROW): now also D60.2 (A)
- net at MX58.2 (ROW): now also D61.2 (A)
- net at MX64.2 (ROW): now also D67.2 (A)
- net at MX73.2 (ROW): now also D76.2 (A)
- net at MX74.2 (ROW): now also D77.2 (A)
- net at MX79.2 (ROW): now also D82.2 (A)
- net at MX80.2 (ROW): now also D83.2 (A)
- net at MX3.2 (ROW): now also D5.2 (A)
- net at MX4.2 (ROW): now also D6.2 (A)
- net at MX6.2 (ROW): now also D8.2 (A)
- net at MX71.2 (ROW): now also D74.2 (A)
- net at MX68.2 (ROW): now also D71.2 (A)
- net at MX5.2 (ROW): now also D7.2 (A)
- net at MX63.2 (ROW): now also D66.2 (A)
- new net Row_10: D50.1 (K), D61.1 (K), D77.1 (K), D8.1 (K)
- new net Row_11: D14.1 (K), D34.1 (K), D67.1 (K), D83.1 (K)
- new net Row_2: D16.1 (K), D25.1 (K), D36.1 (K), D4.1 (K), D46.1 (K), D57.1 (K), D69.1 (K), D75.1 (K)
- new net Row_3: D10.1 (K), D20.1 (K), D30.1 (K), D41.1 (K), D52.1 (K), D63.1 (K), D73.1 (K), D79.1 (K)
- new net Row_4: D17.1 (K), D26.1 (K), D37.1 (K), D47.1 (K), D5.1 (K), D58.1 (K), D70.1 (K), D80.1 (K)
- new net Row_5: D11.1 (K), D21.1 (K), D31.1 (K), D42.1 (K), D53.1 (K), D64.1 (K), D74.1 (K)
- new net Row_6: D18.1 (K), D27.1 (K), D38.1 (K), D48.1 (K), D59.1 (K), D6.1 (K), D71.1 (K)
- new net Row_7: D12.1 (K), D22.1 (K), D32.1 (K), D43.1 (K), D54.1 (K), D65.1 (K), D81.1 (K)
- new net Row_8: D19.1 (K), D28.1 (K), D39.1 (K), D49.1 (K), D60.1 (K), D7.1 (K), D76.1 (K)
- new net Row_9: D13.1 (K), D23.1 (K), D33.1 (K), D44.1 (K), D55.1 (K), D66.1 (K), D82.1 (K)
Other:
- note removed: "Caps"
- note removed: "Ctrl"
- note removed: "Shift"
- note removed: "TAB"
- note removed: "bkspc"
- note removed: "enter"
- moved on the sheet: D3, MX1, MX10, MX11, MX12, MX13, MX14, MX15, MX16, MX17, MX18, MX19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
