File: TKKB-60ish.kicad_pcb (KiCad board)
At the start: 2 copper layers, 24 parts, among them J1 AVR-ISP-6, U1 ATmega32A-PU, Y1 16MHz

Commit message: update to kicad schematic and pcb
Parts:
- added C3: 4u7, Capacitor_THT:CP_Radial_D5.0mm_P2.00mm, F.Cu at (211.9, 350.0)
- added C4: 0u1, Capacitor_THT:C_Disc_D5.1mm_W3.2mm_P5.00mm, F.Cu at (219.1, 350.0)
- added C5: 0u1, Capacitor_THT:C_Disc_D5.1mm_W3.2mm_P5.00mm, F.Cu at (228.6, 350.0)
- added D10: 1N4148TR, Diode_THT:D_DO-35_SOD27_P7.62mm_Horizontal, F.Cu at (241.0, 286.4)
- added D11: 1N4148TR, Diode_THT:D_DO-35_SOD27_P7.62mm_Horizontal, F.Cu at (327.2, 289.9)
- added D12: 1N4148TR, Diode_THT:D_DO-35_SOD27_P7.62mm_Horizontal, F.Cu at (271.3, 266.2)
- added D13: 1N4148TR, Diode_THT:D_DO-35_SOD27_P7.62mm_Horizontal, F.Cu at (271.3, 262.7)
- added D14: 1N4148TR, Diode_THT:D_DO-35_SOD27_P7.62mm_Horizontal, F.Cu at (346.2, 300.8)
- added D15: 1N4148TR, Diode_THT:D_DO-35_SOD27_P7.62mm_Horizontal, F.Cu at (346.2, 297.2)
- added D16: 1N4148TR, Diode_THT:D_DO-35_SOD27_P7.62mm_Horizontal, F.Cu at (316.4, 279.3)
- added D17: 1N4148TR, Diode_THT:D_DO-35_SOD27_P7.62mm_Horizontal, F.Cu at (271.3, 259.1)
- added D18: 1N4148TR, Diode_THT:D_DO-35_SOD27_P7.62mm_Horizontal, F.Cu at (327.2, 286.4)
- added D19: 1N4148TR, Diode_THT:D_DO-35_SOD27_P7.62mm_Horizontal, F.Cu at (327.2, 282.8)
- added D20: 1N4148TR, Diode_THT:D_DO-35_SOD27_P7.62mm_Horizontal, F.Cu at (338.0, 279.3)
- added D21: 1N4148TR, Diode_THT:D_DO-35_SOD27_P7.62mm_Horizontal, F.Cu at (316.4, 289.9)
- added D22: 1N4148TR, Diode_THT:D_DO-35_SOD27_P7.62mm_Horizontal, F.Cu at (327.2, 279.3)
- added D23: 1N4148TR, Diode_THT:D_DO-35_SOD27_P7.62mm_Horizontal, F.Cu at (327.2, 275.7)
- added D24: 1N4148TR, Diode_THT:D_DO-35_SOD27_P7.62mm_Horizontal, F.Cu at (305.7, 289.9)
- added D25: 1N4148TR, Diode_THT:D_DO-35_SOD27_P7.62mm_Horizontal, F.Cu at (316.4, 286.4)
- added D26: 1N4148TR, Diode_THT:D_DO-35_SOD27_P7.62mm_Horizontal, F.Cu at (316.4, 282.8)
- added D27: 1N4148TR, Diode_THT:D_DO-35_SOD27_P7.62mm_Horizontal, F.Cu at (346.2, 293.7)
- added D28: 1N4148TR, Diode_THT:D_DO-35_SOD27_P7.62mm_Horizontal, F.Cu at (176.4, 280.5)
- added D29: 1N4148TR, Diode_THT:D_DO-35_SOD27_P7.62mm_Horizontal, F.Cu at (187.2, 277.0)
- added D3: 1N4148TR, Diode_THT:D_DO-35_SOD27_P7.62mm_Horizontal, F.Cu at (294.9, 289.9)
- added D30: 1N4148TR, Diode_THT:D_DO-35_SOD27_P7.62mm_Horizontal, F.Cu at (273.3, 286.4)
- added D31: 1N4148TR, Diode_THT:D_DO-35_SOD27_P7.62mm_Horizontal, F.Cu at (294.9, 286.4)
- added D32: 1N4148TR, Diode_THT:D_DO-35_SOD27_P7.62mm_Horizontal, F.Cu at (294.9, 282.8)
- added D33: 1N4148TR, Diode_THT:D_DO-35_SOD27_P7.62mm_Horizontal, F.Cu at (294.9, 279.3)
- added D34: 1N4148TR, Diode_THT:D_DO-35_SOD27_P7.62mm_Horizontal, F.Cu at (305.7, 275.7)
- added D35: 1N4148TR, Diode_THT:D_DO-35_SOD27_P7.62mm_Horizontal, F.Cu at (262.6, 286.4)
- added D36: 1N4148TR, Diode_THT:D_DO-35_SOD27_P7.62mm_Horizontal, F.Cu at (284.1, 286.4)
- added D37: 1N4148TR, Diode_THT:D_DO-35_SOD27_P7.62mm_Horizontal, F.Cu at (284.1, 282.8)
- added D38: 1N4148TR, Diode_THT:D_DO-35_SOD27_P7.62mm_Horizontal, F.Cu at (273.3, 289.9)
- added D39: 1N4148TR, Diode_THT:D_DO-35_SOD27_P7.62mm_Horizontal, F.Cu at (284.1, 279.3)
- added D4: 1N4148TR, Diode_THT:D_DO-35_SOD27_P7.62mm_Horizontal, F.Cu at (305.7, 279.3)
- added D40: 1N4148TR, Diode_THT:D_DO-35_SOD27_P7.62mm_Horizontal, F.Cu at (284.1, 275.7)
- added D41: 1N4148TR, Diode_THT:D_DO-35_SOD27_P7.62mm_Horizontal, F.Cu at (284.1, 289.9)
- added D42: 1N4148TR, Diode_THT:D_DO-35_SOD27_P7.62mm_Horizontal, F.Cu at (273.3, 282.8)
- added D43: 1N4148TR, Diode_THT:D_DO-35_SOD27_P7.62mm_Horizontal, F.Cu at (262.6, 289.9)
- added D44: 1N4148TR, Diode_THT:D_DO-35_SOD27_P7.62mm_Horizontal, F.Cu at (273.3, 279.3)
- added D45: 1N4148TR, Diode_THT:D_DO-35_SOD27_P7.62mm_Horizontal, F.Cu at (273.3, 275.7)
- added D46: 1N4148TR, Diode_THT:D_DO-35_SOD27_P7.62mm_Horizontal, F.Cu at (294.9, 275.7)
- added D47: 1N4148TR, Diode_THT:D_DO-35_SOD27_P7.62mm_Horizontal, F.Cu at (348.7, 275.7)
- added D48: 1N4148TR, Diode_THT:D_DO-35_SOD27_P7.62mm_Horizontal, F.Cu at (396.1, 253.3)
- added D49: 1N4148TR, Diode_THT:D_DO-35_SOD27_P7.62mm_Horizontal, F.Cu at (375.9, 273.5)
- added D5: 1N4148TR, Diode_THT:D_DO-35_SOD27_P7.62mm_Horizontal, F.Cu at (305.7, 282.8)
- added D50: 1N4148TR, Diode_THT:D_DO-35_SOD27_P7.62mm_Horizontal, F.Cu at (338.0, 282.8)
- added D51: 1N4148TR, Diode_THT:D_DO-35_SOD27_P7.62mm_Horizontal, F.Cu at (338.0, 275.7)
- added D52: 1N4148TR, Diode_THT:D_DO-35_SOD27_P7.62mm_Horizontal, F.Cu at (262.6, 282.8)
- added D53: 1N4148TR, Diode_THT:D_DO-35_SOD27_P7.62mm_Horizontal, F.Cu at (262.6, 279.3)
- added D54: 1N4148TR, Diode_THT:D_DO-35_SOD27_P7.62mm_Horizontal, F.Cu at (262.6, 275.7)
- added D55: 1N4148TR, Diode_THT:D_DO-35_SOD27_P7.62mm_Horizontal, F.Cu at (251.8, 289.9)
- added D56: 1N4148TR, Diode_THT:D_DO-35_SOD27_P7.62mm_Horizontal, F.Cu at (251.8, 286.4)
- added D57: 1N4148TR, Diode_THT:D_DO-35_SOD27_P7.62mm_Horizontal, F.Cu at (251.8, 282.8)
- added D58: 1N4148TR, Diode_THT:D_DO-35_SOD27_P7.62mm_Horizontal, F.Cu at (241.0, 289.9)
- added D59: 1N4148TR, Diode_THT:D_DO-35_SOD27_P7.62mm_Horizontal, F.Cu at (251.8, 279.3)
- added D6: 1N4148TR, Diode_THT:D_DO-35_SOD27_P7.62mm_Horizontal, F.Cu at (316.4, 275.7)
- added D60: 1N4148TR, Diode_THT:D_DO-35_SOD27_P7.62mm_Horizontal, F.Cu at (219.5, 284.1)
- added D61: 1N4148TR, Diode_THT:D_DO-35_SOD27_P7.62mm_Horizontal, F.Cu at (251.8, 275.7)
- added D62: 1N4148TR, Diode_THT:D_DO-35_SOD27_P7.62mm_Horizontal, F.Cu at (241.0, 282.8)
- added D63: 1N4148TR, Diode_THT:D_DO-35_SOD27_P7.62mm_Horizontal, F.Cu at (230.3, 287.6)
- added D64: 1N4148TR, Diode_THT:D_DO-35_SOD27_P7.62mm_Horizontal, F.Cu at (230.3, 284.1)
- added D65: 1N4148TR, Diode_THT:D_DO-35_SOD27_P7.62mm_Horizontal, F.Cu at (241.0, 279.3)
- added D66: 1N4148TR, Diode_THT:D_DO-35_SOD27_P7.62mm_Horizontal, F.Cu at (241.0, 275.7)
- added D67: 1N4148TR, Diode_THT:D_DO-35_SOD27_P7.62mm_Horizontal, F.Cu at (230.3, 280.5)
- added D68: 1N4148TR, Diode_THT:D_DO-35_SOD27_P7.62mm_Horizontal, F.Cu at (230.3, 277.0)
- added D69: 1N4148TR, Diode_THT:D_DO-35_SOD27_P7.62mm_Horizontal, F.Cu at (219.5, 287.6)
- added D7: 1N4148TR, Diode_THT:D_DO-35_SOD27_P7.62mm_Horizontal, F.Cu at (305.7, 286.4)
- added D70: 1N4148TR, Diode_THT:D_DO-35_SOD27_P7.62mm_Horizontal, F.Cu at (187.2, 280.5)
- added D71: 1N4148TR, Diode_THT:D_DO-35_SOD27_P7.62mm_Horizontal, F.Cu at (176.4, 277.0)
- added D72: 1N4148TR, Diode_THT:D_DO-35_SOD27_P7.62mm_Horizontal, F.Cu at (176.4, 284.1)
- added D73: 1N4148TR, Diode_THT:D_DO-35_SOD27_P7.62mm_Horizontal, F.Cu at (219.5, 280.5)
- added D74: 1N4148TR, Diode_THT:D_DO-35_SOD27_P7.62mm_Horizontal, F.Cu at (219.5, 277.0)
- added D75: 1N4148TR, Diode_THT:D_DO-35_SOD27_P7.62mm_Horizontal, F.Cu at (208.7, 287.6)
- added D76: 1N4148TR, Diode_THT:D_DO-35_SOD27_P7.62mm_Horizontal, F.Cu at (208.7, 284.1)
- added D77: 1N4148TR, Diode_THT:D_DO-35_SOD27_P7.62mm_Horizontal, F.Cu at (208.7, 280.5)
- added D78: 1N4148TR, Diode_THT:D_DO-35_SOD27_P7.62mm_Horizontal, F.Cu at (208.7, 277.0)
- added D79: 1N4148TR, Diode_THT:D_DO-35_SOD27_P7.62mm_Horizontal, F.Cu at (198.0, 287.6)
- added D8: 1N4148TR, Diode_THT:D_DO-35_SOD27_P7.62mm_Horizontal, F.Cu at (187.2, 284.1)
- added D80: 1N4148TR, Diode_THT:D_DO-35_SOD27_P7.62mm_Horizontal, F.Cu at (198.0, 284.1)
- added D81: 1N4148TR, Diode_THT:D_DO-35_SOD27_P7.62mm_Horizontal, F.Cu at (198.0, 280.5)
- added D82: 1N4148TR, Diode_THT:D_DO-35_SOD27_P7.62mm_Horizontal, F.Cu at (176.4, 287.6)
- added D83: 1N4148TR, Diode_THT:D_DO-35_SOD27_P7.62mm_Horizontal, F.Cu at (198.0, 277.0)
- added D9: 1N4148TR, Diode_THT:D_DO-35_SOD27_P7.62mm_Horizontal, F.Cu at (187.2, 287.6)
- added MX10: A, Button_Switch_Keyboard:SW_Cherry_MX_1.00u_PCB, F.Cu at (150.2, 185.4)
- added MX11: Z, Button_Switch_Keyboard:SW_Cherry_MX_1.00u_PCB, F.Cu at (159.7, 204.5)
- added MX12: Alt, Button_Switch_Keyboard:SW_Cherry_MX_1.00u_PCB, F.Cu at (164.5, 223.5)
- added MX13: F2, Button_Switch_Keyboard:SW_Cherry_MX_1.00u_PCB, F.Cu at (169.2, 123.5)
- added MX14: 2, Button_Switch_Keyboard:SW_Cherry_MX_1.00u_PCB, F.Cu at (154.9, 147.3)
- added MX15: W, Button_Switch_Keyboard:SW_Cherry_MX_1.00u_PCB, F.Cu at (164.5, 166.4)
- added MX16: S, Button_Switch_Keyboard:SW_Cherry_MX_1.00u_PCB, F.Cu at (169.2, 185.4)
- added MX17: X, Button_Switch_Keyboard:SW_Cherry_MX_1.00u_PCB, F.Cu at (178.8, 204.5)
- added MX18: 3, Button_Switch_Keyboard:SW_Cherry_MX_1.00u_PCB, F.Cu at (174.0, 147.3)
- added MX19: E, Button_Switch_Keyboard:SW_Cherry_MX_1.00u_PCB, F.Cu at (183.5, 166.4)
- added MX20: D, Button_Switch_Keyboard:SW_Cherry_MX_1.00u_PCB, F.Cu at (188.3, 185.4)
- added MX21: C, Button_Switch_Keyboard:SW_Cherry_MX_1.00u_PCB, F.Cu at (197.8, 204.5)
- added MX22: F3, Button_Switch_Keyboard:SW_Cherry_MX_1.00u_PCB, F.Cu at (188.3, 123.5)
- added MX23: 4, Button_Switch_Keyboard:SW_Cherry_MX_1.00u_PCB, F.Cu at (193.0, 147.3)
- added MX24: R, Button_Switch_Keyboard:SW_Cherry_MX_1.00u_PCB, F.Cu at (202.6, 166.4)
- added MX25: F, Button_Switch_Keyboard:SW_Cherry_MX_1.00u_PCB, F.Cu at (207.3, 185.4)
- added MX26: V, Button_Switch_Keyboard:SW_Cherry_MX_1.00u_PCB, F.Cu at (216.9, 204.5)
- added MX27: F4, Button_Switch_Keyboard:SW_Cherry_MX_1.00u_PCB, F.Cu at (207.3, 123.5)
- added MX28: 5, Button_Switch_Keyboard:SW_Cherry_MX_1.00u_PCB, F.Cu at (212.1, 147.3)
- added MX29: T, Button_Switch_Keyboard:SW_Cherry_MX_1.00u_PCB, F.Cu at (221.6, 166.4)
- added MX30: G, Button_Switch_Keyboard:SW_Cherry_MX_1.00u_PCB, F.Cu at (226.4, 185.4)
- added MX31: B, Button_Switch_Keyboard:SW_Cherry_MX_1.00u_PCB, F.Cu at (235.9, 204.5)
- added MX32: F5, Button_Switch_Keyboard:SW_Cherry_MX_1.00u_PCB, F.Cu at (235.9, 123.5)
- added MX33: 6, Button_Switch_Keyboard:SW_Cherry_MX_1.00u_PCB, F.Cu at (231.1, 147.3)
- added MX34: Y, Button_Switch_Keyboard:SW_Cherry_MX_1.00u_PCB, F.Cu at (240.7, 166.4)
- added MX35: H, Button_Switch_Keyboard:SW_Cherry_MX_1.00u_PCB, F.Cu at (245.4, 185.4)
- added MX36: N, Button_Switch_Keyboard:SW_Cherry_MX_1.00u_PCB, F.Cu at (255.0, 204.5)
- added MX37: F6, Button_Switch_Keyboard:SW_Cherry_MX_1.00u_PCB, F.Cu at (255.0, 123.5)
- added MX38: 7, Button_Switch_Keyboard:SW_Cherry_MX_1.00u_PCB, F.Cu at (250.2, 147.3)
- added MX39: U, Button_Switch_Keyboard:SW_Cherry_MX_1.00u_PCB, F.Cu at (259.7, 166.4)
- added MX40: J, Button_Switch_Keyboard:SW_Cherry_MX_1.00u_PCB, F.Cu at (264.5, 185.4)
- added MX41: M, Button_Switch_Keyboard:SW_Cherry_MX_1.00u_PCB, F.Cu at (274.0, 204.5)
- added MX42: F7, Button_Switch_Keyboard:SW_Cherry_MX_1.00u_PCB, F.Cu at (274.0, 123.5)
- added MX43: 8, Button_Switch_Keyboard:SW_Cherry_MX_1.00u_PCB, F.Cu at (269.2, 147.3)
- added MX44: I, Button_Switch_Keyboard:SW_Cherry_MX_1.00u_PCB, F.Cu at (278.8, 166.4)
- added MX45: K, Button_Switch_Keyboard:SW_Cherry_MX_1.00u_PCB, F.Cu at (283.5, 185.4)
- added MX46: <, Button_Switch_Keyboard:SW_Cherry_MX_1.00u_PCB, F.Cu at (293.1, 204.5)
- added MX47: R Alt, Button_Switch_Keyboard:SW_Cherry_MX_1.00u_PCB, F.Cu at (316.9, 223.5)
- added MX48: F8, Button_Switch_Keyboard:SW_Cherry_MX_1.00u_PCB, F.Cu at (293.1, 123.5)
- added MX49: 9, Button_Switch_Keyboard:SW_Cherry_MX_1.00u_PCB, F.Cu at (288.3, 147.3)
- added MX50: O, Button_Switch_Keyboard:SW_Cherry_MX_1.00u_PCB, F.Cu at (297.8, 166.4)
- added MX51: L, Button_Switch_Keyboard:SW_Cherry_MX_1.00u_PCB, F.Cu at (302.6, 185.4)
- added MX52: >, Button_Switch_Keyboard:SW_Cherry_MX_1.00u_PCB, F.Cu at (312.1, 204.5)
- added MX53: F9, Button_Switch_Keyboard:SW_Cherry_MX_1.00u_PCB, F.Cu at (321.6, 123.5)
- added MX54: 0, Button_Switch_Keyboard:SW_Cherry_MX_1.00u_PCB, F.Cu at (307.3, 147.3)
- added MX55: P, Button_Switch_Keyboard:SW_Cherry_MX_1.00u_PCB, F.Cu at (316.9, 166.4)
- added MX56: ;, Button_Switch_Keyboard:SW_Cherry_MX_1.00u_PCB, F.Cu at (321.6, 185.4)
- added MX57: /, Button_Switch_Keyboard:SW_Cherry_MX_1.00u_PCB, F.Cu at (331.2, 204.5)
- added MX58: R Ctrl, Button_Switch_Keyboard:SW_Cherry_MX_1.00u_PCB, F.Cu at (335.9, 223.5)
- added MX59: F10, Button_Switch_Keyboard:SW_Cherry_MX_1.00u_PCB, F.Cu at (340.7, 123.5)
- added MX60: -, Button_Switch_Keyboard:SW_Cherry_MX_1.00u_PCB, F.Cu at (326.4, 147.3)
- added MX61: [, Button_Switch_Keyboard:SW_Cherry_MX_1.00u_PCB, F.Cu at (335.9, 166.4)
- added MX62: ', Button_Switch_Keyboard:SW_Cherry_MX_1.00u_PCB, F.Cu at (340.7, 185.4)
- added MX63: RShift, Button_Switch_Keyboard:SW_Cherry_MX_1.75u_PCB, F.Cu at (357.3, 204.5)
- added MX64: Left Arrow, Button_Switch_Keyboard:SW_Cherry_MX_1.00u_PCB, F.Cu at (364.5, 223.5)
- added MX65: F11, Button_Switch_Keyboard:SW_Cherry_MX_1.00u_PCB, F.Cu at (359.7, 123.5)
- added MX66: =, Button_Switch_Keyboard:SW_Cherry_MX_1.00u_PCB, F.Cu at (345.4, 147.3)
- added MX67: ], Button_Switch_Keyboard:SW_Cherry_MX_1.00u_PCB, F.Cu at (355.0, 166.4)
- added MX68: Enter, Button_Switch_Keyboard:SW_Cherry_MX_2.25u_PCB, F.Cu at (366.6, 195.6)
- added MX69: F12, Button_Switch_Keyboard:SW_Cherry_MX_1.00u_PCB, F.Cu at (378.8, 123.5)
- added MX70: \, Button_Switch_Keyboard:SW_Cherry_MX_1.00u_PCB, F.Cu at (364.5, 147.3)
- added MX71: bACKSPACE, Button_Switch_Keyboard:SW_Cherry_MX_1.50u_PCB, F.Cu at (378.8, 166.4)
- added MX72: Del, Button_Switch_Keyboard:SW_Cherry_MX_1.00u_PCB, F.Cu at (383.5, 147.3)
- added MX73: Up Arrow, Button_Switch_Keyboard:SW_Cherry_MX_1.00u_PCB, F.Cu at (383.5, 204.5)
- added MX74: Down Arrow, Button_Switch_Keyboard:SW_Cherry_MX_1.00u_PCB, F.Cu at (383.5, 223.5)
- added MX75: ?, Button_Switch_Keyboard:SW_Cherry_MX_1.00u_PCB, F.Cu at (402.6, 123.5)
- added MX76: Home, Button_Switch_Keyboard:SW_Cherry_MX_1.00u_PCB, F.Cu at (402.6, 147.3)
- added MX77: PgUp, Button_Switch_Keyboard:SW_Cherry_MX_1.00u_PCB, F.Cu at (402.6, 166.4)
- added MX78: PgDn, Button_Switch_Keyboard:SW_Cherry_MX_1.00u_PCB, F.Cu at (402.6, 185.4)
- added MX79: End, Button_Switch_Keyboard:SW_Cherry_MX_1.00u_PCB, F.Cu at (402.6, 204.5)
- added MX80: Right Arrow, Button_Switch_Keyboard:SW_Cherry_MX_1.00u_PCB, F.Cu at (402.6, 223.5)
- added MX9: Q, Button_Switch_Keyboard:SW_Cherry_MX_1.00u_PCB, F.Cu at (145.4, 166.4)
- MX1: value MX-NoLED -> Esc
- MX2: value MX-NoLED -> Tilde
- MX3: value MX-NoLED -> Tab; footprint Button_Switch_Keyboard:SW_Cherry_MX_1.00u_PCB -> Button_Switch_Keyboard:SW_Cherry_MX_1.50u_PCB
- MX4: value MX-NoLED -> Step Caps
- MX5: value MX-NoLED -> Shift; footprint Button_Switch_Keyboard:SW_Cherry_MX_1.00u_PCB -> Button_Switch_Keyboard:SW_Cherry_MX_2.25u_PCB
- MX6: value MX-NoLED -> Ctrl; footprint Button_Switch_Keyboard:SW_Cherry_MX_1.00u_PCB -> Button_Switch_Keyboard:SW_Cherry_MX_1.50u_PCB
- MX7: value MX-NoLED -> F1
- MX8: value MX-NoLED -> 1
- moved J1 280.8 mm to (228.6, 359.6), turned to 0 degrees
- moved C1 274.6 mm to (285.8, 378.6), turned to 0 degrees
- moved C2 272.4 mm to (307.2, 378.6)
- moved Y1 271.6 mm to (295.3, 378.6), turned to 0 degrees
- moved D2 266.6 mm to (266.7, 371.5)
- moved D1 263.9 mm to (266.7, 364.3)
- moved R3 260.6 mm to (285.8, 359.6), turned to 0 degrees
- moved R5 259.0 mm to (285.8, 369.1), turned to 0 degrees
- moved R4 254.0 mm to (285.8, 364.3), turned to 0 degrees
- moved R2 251.8 mm to (285.8, 354.8), turned to 0 degrees
- moved Boot1 251.3 mm to (226.2, 336.0), turned to 0 degrees
- moved R1 247.1 mm to (285.8, 350.0), turned to 0 degrees
- moved U1 237.4 mm to (240.7, 323.8), turned to 0 degrees
- moved F1 236.9 mm to (285.8, 342.9), turned to 0 degrees
- moved Reset1 236.6 mm to (226.2, 324.1), turned to 0 degrees
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Connections:
- net Net-(U1-Pad1) renamed Row_0
- net Net-(U1-Pad2) renamed Row_1
- net Net-(U1-Pad22) renamed Row_5
- net Net-(U1-Pad23) renamed Row_6
- net Net-(U1-Pad24) renamed Row_7
- net Net-(U1-Pad25) renamed Row_8
- net Net-(U1-Pad26) renamed Row_9
- net Net-(U1-Pad27) renamed Row_10
- net Net-(U1-Pad28) renamed Row_11
- net Net-(U1-Pad3) renamed Row_2
- net Net-(U1-Pad33) renamed Col_7
- net Net-(U1-Pad34) renamed Col_6
- net Net-(U1-Pad35) renamed Col_5
- net Net-(U1-Pad36) renamed Col_4
- net Net-(U1-Pad37) renamed Col_3
- net Net-(U1-Pad38) renamed Col_2
- net Net-(U1-Pad39) renamed Col_1
- net Net-(U1-Pad4) renamed Row_3
- net Net-(U1-Pad40) renamed Col_0
- net Net-(U1-Pad5) renamed Row_4
- MX1 pad 1: Net-(MX1-Pad1) -> /Keyboard Matrix/Col_0
- MX2 pad 1: Net-(MX2-Pad1) -> /Keyboard Matrix/Col_0
- MX3 pad 1: Net-(MX3-Pad1) -> /Keyboard Matrix/Col_0
- MX4 pad 1: Net-(MX4-Pad1) -> /Keyboard Matrix/Col_0
- MX5 pad 1: Net-(MX5-Pad1) -> /Keyboard Matrix/Col_0
- MX6 pad 1: Net-(MX6-Pad1) -> /Keyboard Matrix/Col_0
- MX7 pad 1: Net-(MX7-Pad1) -> /Keyboard Matrix/Col_0
- MX8 pad 1: Net-(MX8-Pad1) -> /Keyboard Matrix/Col_0
- R1 pad 2: USB_CC -> GND
- R2 pad 2: USB_CC -> GND

Commit message: Board layout work
Parts:
- moved D14 290.7 mm to (135.1, 101.0), turned to 90 degrees
- moved D15 278.5 mm to (138.5, 111.8), turned to 90 degrees
- moved D11 270.9 mm to (127.3, 107.0), turned to 90 degrees
- moved D6 264.5 mm to (113.6, 105.9), turned to 90 degrees
- moved D7 263.1 mm to (116.2, 103.8), turned to 90 degrees
- moved D5 261.7 mm to (111.0, 107.9), turned to 90 degrees
- moved D4 260.0 mm to (108.4, 109.8), turned to 90 degrees
- moved D3 259.8 mm to (105.8, 111.8), turned to 90 degrees
- moved D18 255.6 mm to (146.3, 105.8), turned to 90 degrees
- moved D19 252.6 mm to (148.9, 103.9), turned to 90 degrees
- moved D20 250.2 mm to (154.5, 109.2), turned to 90 degrees
- moved USB1 244.9 mm to (123.5, 342.4)
- moved D16 243.8 mm to (141.1, 109.8), turned to 90 degrees
- moved D21 242.3 mm to (157.1, 107.3), turned to 90 degrees
- moved D12 214.4 mm to (129.9, 105.0), turned to 90 degrees
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Routing:
- net /Keyboard Matrix/Col_1: track 0.00 -> 1.56 mm
